Commit message: 1

File: description/target.urdf.xacro (robot description, xacro)
@@ -3,7 +3,7 @@
     <xacro:include filename="target_core.xacro" />
     <!-- <xacro:include filename="gazebo_control.xacro"/> -->
-    <!-- <xacro:include filename="ros2_control.xacro"/>
-    <xacro:include filename="lidar.xacro"/>
-    <xacro:include filename="camera.xacro"/>
-    <xacro:include filename="depth_camera.xacro"/> -->
+    <xacro:include filename="target_control.xacro"/>
+    <!-- <xacro:include filename="lidar.xacro"/> -->
+    <!-- <xacro:include filename="camera.xacro"/> -->
+    <!-- <xacro:include filename="depth_camera.xacro"/> -->
 </robot>

File: description/target_control.xacro (robot description, xacro)
@@ -6,5 +6,5 @@
             <plugin>gazebo_ros2_control/GazeboSystem</plugin>
         </hardware>
-        <joint name="base_left_wheel_joint">
+        <joint name="sphere_left_wheel_joint">
             <!-- command interfaces -->
             <command_interface name="velocity">
@@ -16,5 +16,5 @@
             <state_interface name="position" />
         </joint>
-        <joint name="base_right_wheel_joint">
+        <joint name="sphere_right_wheel_joint">
             <!-- command interfaces -->
             <command_interface name="velocity">
@@ -30,8 +30,8 @@
         <plugin name="gazebo_ros2_control" filename="libgazebo_ros2_control.so">
             <ros>
-                <namespace>robot</namespace>
+                <namespace>target</namespace>
                 <remapping>/robot_description:=/robot_description_full</remapping>
             </ros>
-            <parameters>/home/nusshao/dev_ws/src/tracking_project/config/my_controllers.yaml</parameters>
+            <parameters>/home/nusshao/dev_ws/src/tracking_project/config/target_controllers.yaml</parameters>
         </plugin>
     </gazebo>

File: description/target_core.xacro (robot description, xacro)
@@ -2,6 +2,10 @@
 <robot xmlns:xacro="http://www.ros.org/wiki/xacro">
     <xacro:include filename="inertial_macros.xacro" />
+    <!-- <xacro:property name="tf_prefix" value="target/" /> -->
     <material name="orange">
         <color rgba="1 0.3 0.1 1" />
+    </material>
+    <material name="black">
+        <color rgba="0.1 0.1 0.1 1" />
     </material>
     <!-- base link -->
@@ -13,5 +17,5 @@
         <parent link="base_link" />
         <child link="sphere_link" />
-        <origin xyz="0 0 0.1" />
+        <origin xyz="0 0 0" />
     </joint>
     <link name="sphere_link">
@@ -33,6 +37,55 @@
     <gazebo reference="sphere_link">
         <material>Gazebo/Orange</material>
-        <mu1 value="0.001" />
-        <mu2 value="0.001" />
+    </gazebo>
+    <!-- left wheel link -->
+    <joint name="sphere_left_wheel_joint" type="continuous">
+        <parent link="base_link" />
+        <child link="left_wheel_link" />
+        <origin xyz="0 0.22 0" rpy="-${pi/2} 0 0" />
+        <axis xyz="0 0 1" />
+    </joint>
+    <link name="left_wheel_link">
+        <visual>
+            <geometry>
+                <cylinder radius="0.22" length="0.04" />
+            </geometry>
+            <material name="black" />
+        </visual>
+        <collision>
+            <geometry>
+                <cylinder radius="0.22" length="0.04" />
+            </geometry>
+        </collision>
+        <xacro:inertial_cylinder mass="0.5" length="0.04" radius="0.22">
+            <origin xyz="0 0 0" rpy="0 0 0" />
+        </xacro:inertial_cylinder>
+    </link>
+    <gazebo reference="left_wheel_link">
+        <material>Gazebo/Black</material>
+    </gazebo>
+    <joint name="sphere_right_wheel_joint" type="continuous">
+        <parent link="base_link" />
+        <child link="right_wheel_link" />
+        <origin xyz="0 -0.22 0" rpy="${pi/2} 0 0" />
+        <axis xyz="0 0 -1" />
+    </joint>
+    <link name="right_wheel_link">
+        <visual>
+            <geometry>
+                <cylinder radius="0.22" length="0.04" />
+            </geometry>
+            <material name="black" />
+        </visual>
+        <collision>
+            <geometry>
+                <cylinder radius="0.22" length="0.04" />
+            </geometry>
+        </collision>
+        <xacro:inertial_cylinder mass="0.5" length="0.04" radius="0.22">
+            <origin xyz="0 0 0" rpy="0 0 0" />
+        </xacro:inertial_cylinder>
+    </link>
+    <gazebo reference="right_wheel_link">
+        <material>Gazebo/Black</material>
     </gazebo>
 </robot>
