Commit message: 1

File: description/target_core.xacro (robot description, xacro)
@@ -89,3 +89,55 @@
         <material>Gazebo/Black</material>
     </gazebo>
+    <joint name="sphere_first_bar_joint" type="fixed">
+        <parent link="right_wheel_link" />
+        <child link="first_bar_link" />
+        <origin xyz="0 0 0.2" />
+    </joint>
+    <link name="first_bar_link">
+        <visual>
+            <geometry>
+                <box size="0.04 0.42 0.005" />
+            </geometry>
+            <material name="black" />
+            <origin xyz="0 0.2 -0.42" rpy="-${pi/2} 0 0"/>
+        </visual>
+        <collision>
+            <geometry>
+                <box size="0.04 0.42 0.005" />
+            </geometry>
+            <origin xyz="0 0 0" />
+        </collision>
+        <xacro:inertial_box mass="0.001" x="0.04" y="0.42" z="0.005">
+            <origin xyz="0 0 0" rpy="0 0 0" />
+        </xacro:inertial_box>
+    </link>
+    <gazebo reference="first_bar_link">
+        <material>Gazebo/Gray</material>
+    </gazebo>
+    <joint name="sphere_second_bar_joint" type="fixed">
+        <parent link="right_wheel_link" />
+        <child link="second_bar_link" />
+        <origin xyz="0 0 -0.24" />
+    </joint>
+    <link name="second_bar_link">
+        <visual>
+            <geometry>
+                <box size="0.04 0.42 0.005" />
+            </geometry>
+            <material name="black" />
+            <origin xyz="0 -0.2 0" rpy="-${pi/2} 0 0"/>
+        </visual>
+        <collision>
+            <geometry>
+                <box size="0.04 0.42 0.005" />
+            </geometry>
+            <origin xyz="0 0 0" />
+        </collision>
+        <xacro:inertial_box mass="0.001" x="0.04" y="0.42" z="0.005">
+            <origin xyz="0 0 0" rpy="0 0 0" />
+        </xacro:inertial_box>
+    </link>
+    <gazebo reference="second_bar_link">
+        <material>Gazebo/Gray</material>
+    </gazebo>
 </robot>
