Commit message: 1

File: description/robot_core.xacro (robot description, xacro)
@@ -54,4 +54,8 @@
         <origin xyz="0 0.175 0" rpy="-${pi/2} 0 0" />
         <axis xyz="0 0 1" />
+        <!-- <transmission>
+            <type>hardware_interface/VelocityJointInterface</type>
+            <joint name="base_left_wheel_joint"/>
+        </transmission> -->
     </joint>
     <link name="left_wheel_link">
@@ -80,4 +84,8 @@
             <origin xyz="0 -0.175 0" rpy="${pi/2} 0 0" />
             <axis xyz="0 0 -1" />
+            <!-- <transmission>
+                <type>hardware_interface/VelocityJointInterface</type>
+                <joint name="base_left_wheel_joint"/>
+            </transmission> -->
         </joint>
         <link name="right_wheel_link">

File: description/ros2_control.xacro (robot description, xacro)
@@ -34,4 +34,6 @@
             </ros>
             <parameters>/home/nusshao/dev_ws/src/tracking_project/config/my_controllers.yaml</parameters>
+            <!-- robot_param_node is necessory for multi-robot controller declaration!!! -->
+            <robot_param_node>/robot/robot_state_publisher</robot_param_node>
         </plugin>
     </gazebo>

File: description/target_control.xacro (robot description, xacro)
@@ -34,4 +34,6 @@
             </ros>
             <parameters>/home/nusshao/dev_ws/src/tracking_project/config/target_controllers.yaml</parameters>
+            <!-- robot_param_node is necessory for multi-robot controller declaration!!! -->
+            <robot_param_node>/target/robot_state_publisher</robot_param_node>
         </plugin>
     </gazebo>
