Commit message: 1.Image catching python function added. 2.Self-made dataset uploaded.

File: description/camera.xacro (robot description, xacro)
@@ -46,4 +46,7 @@
             <!-- gazebo camera control plugin -->
             <plugin name="camera_controller" filename="libgazebo_ros_camera.so">
+                <ros>
+                    <namespace>robot</namespace>
+                </ros>
                 <frame_name>camera_link_optical</frame_name>
             </plugin>

File: description/target_core.xacro (robot description, xacro)
@@ -63,4 +63,6 @@
     <gazebo reference="left_wheel_link">
         <material>Gazebo/Black</material>
+        <mu1 value="0.1" />
+        <mu2 value="0.1" />
     </gazebo>
     <joint name="sphere_right_wheel_joint" type="continuous">
@@ -88,56 +90,6 @@
     <gazebo reference="right_wheel_link">
         <material>Gazebo/Black</material>
-    </gazebo>
-    <joint name="sphere_first_bar_joint" type="fixed">
-        <parent link="right_wheel_link" />
-        <child link="first_bar_link" />
-        <origin xyz="0 0 0.2" />
-    </joint>
-    <link name="first_bar_link">
-        <visual>
-            <geometry>
-                <box size="0.04 0.42 0.005" />
-            </geometry>
-            <material name="black" />
-            <origin xyz="0 0.2 -0.42" rpy="-${pi/2} 0 0"/>
-        </visual>
-        <collision>
-            <geometry>
-                <box size="0.04 0.42 0.005" />
-            </geometry>
-            <origin xyz="0 0 0" />
-        </collision>
-        <xacro:inertial_box mass="0.001" x="0.04" y="0.42" z="0.005">
-            <origin xyz="0 0 0" rpy="0 0 0" />
-        </xacro:inertial_box>
-    </link>
-    <gazebo reference="first_bar_link">
-        <material>Gazebo/Gray</material>
-    </gazebo>
-    <joint name="sphere_second_bar_joint" type="fixed">
-        <parent link="right_wheel_link" />
-        <child link="second_bar_link" />
-        <origin xyz="0 0 -0.24" />
-    </joint>
-    <link name="second_bar_link">
-        <visual>
-            <geometry>
-                <box size="0.04 0.42 0.005" />
-            </geometry>
-            <material name="black" />
-            <origin xyz="0 -0.2 0" rpy="-${pi/2} 0 0"/>
-        </visual>
-        <collision>
-            <geometry>
-                <box size="0.04 0.42 0.005" />
-            </geometry>
-            <origin xyz="0 0 0" />
-        </collision>
-        <xacro:inertial_box mass="0.001" x="0.04" y="0.42" z="0.005">
-            <origin xyz="0 0 0" rpy="0 0 0" />
-        </xacro:inertial_box>
-    </link>
-    <gazebo reference="second_bar_link">
-        <material>Gazebo/Gray</material>
+        <mu1 value="0.5" />
+        <mu2 value="0.5" />
     </gazebo>
 </robot>

Commit message: New robot model updated

File: description/camera.xacro (robot description, xacro)
@@ -9,5 +9,6 @@
         <visual>
             <geometry>
-                <box size="0.01 0.03 0.03" />
+                <mesh filename='/home/nusshao/dev_ws/src/tracking_project/description/camera.dae' scale='3 3 3'/>
+                <!-- <box size="0.01 0.03 0.03" /> -->
             </geometry>
             <material name="red" />
@@ -22,5 +23,5 @@
     <gazebo reference="camera_link">
         <!-- Color definition in Gazebo -->
-        <material>Gazebo/Red</material>
+        <!-- <material>Gazebo/Red</material> -->
         <!-- Sensor tag for camera -->
         <sensor name="camera" type="camera">

File: description/lidar.xacro (robot description, xacro)
@@ -4,10 +4,11 @@
         <parent link="chassis_link" />
         <child link="laser_frame" />
-        <origin xyz="0.1 0 0.175" rpy="0 0 0" />
+        <origin xyz="0.1 0 0.165" rpy="0 0 0" />
     </joint>
     <link name="laser_frame">
         <visual>
             <geometry>
-                <cylinder radius="0.05" length="0.04" />
+                <mesh filename='/home/nusshao/dev_ws/src/tracking_project/description/lidar.dae' scale='1 1 1'/>
+                <!-- <cylinder radius="0.05" length="0.04" /> -->
             </geometry>
             <material name="red" />
@@ -24,5 +25,5 @@
     <gazebo reference="laser_frame">
         <!-- Color definition in Gazebo -->
-        <material>Gazebo/Red</material>
+        <!-- <material>Gazebo/Red</material> -->
         <!-- ray type sensor -->
         <sensor name="laser" type="ray">

File: description/robot.urdf.xacro (robot description, xacro)
@@ -4,5 +4,5 @@
     <!-- <xacro:include filename="gazebo_control.xacro"/> -->
     <xacro:include filename="ros2_control.xacro"/>
-    <!-- <xacro:include filename="lidar.xacro"/> -->
+    <xacro:include filename="lidar.xacro"/>
     <xacro:include filename="camera.xacro"/>
     <!-- <xacro:include filename="depth_camera.xacro"/> -->

File: description/robot_core.xacro (robot description, xacro)
@@ -29,6 +29,7 @@
     <link name="chassis_link">
         <visual>
-            <geometry>
-                <box size="0.3 0.3 0.15" />
+            <geometry>  <!-- <color sid="emission"> has to be equal to <color sid="diffuse"> -->
+                <mesh filename='/home/nusshao/dev_ws/src/tracking_project/description/chassis.dae' scale='1 1 1'/>
+                <!-- <box size="0.3 0.3 0.15" /> -->
             </geometry>
             <material name="white" />
@@ -62,5 +63,6 @@
         <visual>
             <geometry>
-                <cylinder radius="0.05" length="0.04" />
+                <mesh filename='/home/nusshao/dev_ws/src/tracking_project/description/wheel.dae' scale='1 1 1'/>
+                <!-- <cylinder radius="0.05" length="0.04" /> -->
             </geometry>
             <material name="blue" />
@@ -76,5 +78,5 @@
     </link>
     <gazebo reference="left_wheel_link">
-        <material>Gazebo/Blue</material>
+        <!-- <material>Gazebo/Blue</material> -->
     </gazebo>
         <!-- right wheel link -->
@@ -92,5 +94,6 @@
             <visual>
                 <geometry>
-                    <cylinder radius="0.05" length="0.04" />
+                    <mesh filename='/home/nusshao/dev_ws/src/tracking_project/description/wheel.dae' scale='1 1 1'/>
+                    <!-- <cylinder radius="0.05" length="0.04" /> -->
                 </geometry>
                 <material name="blue" />
@@ -106,5 +109,5 @@
         </link>
         <gazebo reference="right_wheel_link">
-            <material>Gazebo/Blue</material>
+            <!-- <material>Gazebo/Blue</material> -->
         </gazebo>
         <!-- caster wheel link -->
